File: meterkast.kicad_sch (KiCad schematic)
At the start: 23 parts

Commit message: Oplaadpunt Auto
Parts:
- added J?: 0, symbol Connector:Conn_01x01_Male
Connections:
- net at CB?.1: now also J?.1 (Pin_1)
Other:
- note added: "Oplaadpunt Auto"
Changed lines of the file:
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@@
+    (stroke (width 0) (type default) (color 0 0 0 0))
+  )
+  (wire (pts (xy 114.3 144.78) (xy 114.3 149.86))
+    (stroke (width 0) (type default) (color 0 0 0 0))
+  )
+  (wire (pts (xy 163.83 144.78) (xy 114.3 144.78))
     (stroke (width 0) (type default) (color 0 0 0 0))
   )
@@
   )
   (text "Aanrecht keuken" (at 152.4 119.38 90)
+    (effects (font (size 1.27 1.27)) (justify left bottom))
+  )
+  (text "Oplaadpunt Auto" (at 163.83 140.97 0)
     (effects (font (size 1.27 1.27)) (justify left bottom))
   )
@@
     (pin "2")
   )
+  (symbol (lib_id "Connector:Conn_01x01_Male") (at 168.91 144.78 180) (unit 1)
+    (in_bom yes) (on_board yes)
+    (property "Reference" "J?" (id 0) (at 167.64 146.05 90)
+      (effects (font (size 1.27 1.27)) (justify left) hide)
+    )
+    (property "Value" "0" (id 1) (at 166.37 146.05 90)
+      (effects (font (size 1.27 1.27)) (justify left) hide)
+    )
+    (property "Footprint" "" (id 2) (at 168.91 144.78 0)
+      (effects (font (size 1.27 1.27)) hide)
+    )
+    (property "Datasheet" "~" (id 3) (at 168.91 144.78 0)
+      (effects (font (size 1.27 1.27)) hide)
+    )
+    (pin "1")
+  )
   (sheet_instances
     (path "/" (page "1"))
@@
       (reference "J?") (unit 1) (value "7") (footprint "")
     )
+    (path "/9671d64b-da41-48fe-bd9c-062ec19cf730"
+      (reference "J?") (unit 1) (value "0") (footprint "")
+    )
     (path "/00000000-0000-0000-0000-00005e00b3e3"
